Commit message: Fall Robot

File: urdf/Robot_URDF.xacro (robot description, xacro)
@@ -388,5 +388,5 @@
   <joint
     name="Cover_Joint"
-    type="continuous">
+         type="fixed">
     <origin
       xyz="0 0 0"
@@ -396,6 +396,6 @@
     <child
       link="Cover_Link" />
-    <axis
-      xyz="0 0 1" />
+      <!--  <axis
+			xyz="0 0 1" />-->
   </joint>
   <link
@@ -446,10 +446,10 @@
       link="Lidar_Link" />
     <axis
-      xyz="0 0 1" />
-    <limit
+      xyz="0 0 0" />
+   <!-- <limit
       lower="0"
       upper="0"
       effort="0"
-      velocity="0" />
+      velocity="0" /> -->
   </joint>
 </robot>

Commit message: one step left

File: urdf/Robot_URDF.xacro (robot description, xacro)
@@ -417,5 +417,5 @@
     <visual>
       <origin
-        xyz="0 0 0"
+        xyz="0 0 -0.1"
         rpy="0 0 0" />
       <geometry>
@@ -427,5 +427,5 @@
     <collision>
       <origin
-        xyz="0 0 0"
+        xyz="0 0 -0.1"
         rpy="0 0 0" />
       <geometry>
@@ -439,8 +439,8 @@
     type="fixed">
     <origin
-      xyz="0 0 0"
-      rpy="0 0 0" />
-    <parent
-      link="Cover_Link" />
+      xyz="0 0 0.1"
+      rpy="0 0 0" />
+    <parent
+      link="base_link" />
     <child
       link="Lidar_Link" />

Commit message: error at the launch file

File: urdf/Robot_URDF.xacro (robot description, xacro)
@@ -10,4 +10,12 @@
 <!-- Import all Gazebo-customization elements, including Gazebo colors -->
   <xacro:include filename="$(find Robot_URDF)/urdf/mybot.gazebo" />
+        <link name="world"/>
+        <joint name="dummy_joint" type="fixed">
+          <origin xyz="0.0 0.0 0.0" rpy="0.0 0.0 0.0"/>
+          <parent link="world"/>
+          <child link="base_link"/>
+          <axis xyz="0.0 0.0 0.0"/>
+          <limit lower="0.0" upper="0.0" effort="0.0" velocity="0.0"/>
+        </joint>
   <link
     name="base_link">

Commit message: sorting the codes

File: urdf/Robot_URDF.xacro (robot description, xacro)
@@ -10,8 +10,9 @@
 <!-- Import all Gazebo-customization elements, including Gazebo colors -->
   <xacro:include filename="$(find Robot_URDF)/urdf/mybot.gazebo" />
-        <link name="world"/>
+ <!--dummy link-->
+        <link name="base_footprint"/>
         <joint name="dummy_joint" type="fixed">
           <origin xyz="0.0 0.0 0.0" rpy="0.0 0.0 0.0"/>
-          <parent link="world"/>
+          <parent link="base_footprint"/>
           <child link="base_link"/>
           <axis xyz="0.0 0.0 0.0"/>
